Commit message: basic_autonomous_traversal_of_path_working.

File: lhd_description/urdf/lhd.urdf.xacro (robot description, xacro)
@@ -26,5 +26,5 @@
         </visual>
         <collision>
-            <origin xyz="0 0 0" rpy="0 0 0" />
+            <origin xyz="0 0.019 0" rpy="0 0 0" />
             <geometry>
                 <mesh filename="package://lhd_description/meshes/base_link.STL" />
@@ -80,8 +80,14 @@
             </material>
         </visual>
-        <collision>
+        <!-- <collision>
             <origin xyz="0 0 0" rpy="0 0 0" />
             <geometry>
                 <mesh filename="package://lhd_description/meshes/blw.STL" />
+            </geometry>
+        </collision> -->
+        <collision>
+            <origin xyz="0.0 0.0 -0.029" rpy="0.0 0.0 0.0"/>
+            <geometry>
+                <cylinder radius="0.107" length="0.05"/>
             </geometry>
         </collision>
@@ -110,8 +116,14 @@
             </material>
         </visual>
-        <collision>
+        <!-- <collision>
             <origin xyz="0 0 0" rpy="0 0 0" />
             <geometry>
                 <mesh filename="package://lhd_description/meshes/brw.STL" />
+            </geometry>
+        </collision> -->
+        <collision>
+            <origin xyz="0.0 0.0 -0.029" rpy="0.0 0.0 0.0"/>
+            <geometry>
+                <cylinder radius="0.107" length="0.05"/>
             </geometry>
         </collision>
@@ -230,8 +242,14 @@
             </material>
         </visual>
-        <collision>
+        <!-- <collision>
             <origin xyz="0 0 0" rpy="0 0 0" />
             <geometry>
                 <mesh filename="package://lhd_description/meshes/flw.STL" />
+            </geometry>
+        </collision> -->
+        <collision>
+            <origin xyz="0.0 0.0 -0.029" rpy="0.0 0.0 0.0"/>
+            <geometry>
+                <cylinder radius="0.107" length="0.05"/>
             </geometry>
         </collision>
@@ -258,8 +276,14 @@
             </material>
         </visual>
-        <collision>
+        <!-- <collision>
             <origin xyz="0 0 0" rpy="0 0 0" />
             <geometry>
                 <mesh filename="package://lhd_description/meshes/frw.STL" />
+            </geometry>
+        </collision> -->
+        <collision>
+            <origin xyz="0.0 0.0 -0.029" rpy="0.0 0.0 0.0"/>
+            <geometry>
+                <cylinder radius="0.107" length="0.05"/>
             </geometry>
         </collision>
